Commit message: Update 01-myfirst.urdf

File: first_time/urdf/01-myfirst.urdf (robot description, URDF)
Before this commit: robot fourwheelrobot, 5 links, 4 joints
Links:
- added link base_footprint
Joints:
- added joint base_footprint_joint: type fixed, parent base_footprint, child base_link

Commit message: h

File: first_time/urdf/01-myfirst.urdf (robot description, URDF)
Before this commit: robot fourwheelrobot, 6 links, 5 joints
Links:
- link base_link: geometry collision box size=1 0.5 0.2; visual box size=1 0.5 0.2
- link wheel1: geometry collision cylinder length=0.1 radius=0.1; visual cylinder length=0.1 radius=0.1
- link wheel2: geometry collision cylinder length=0.1 radius=0.1; visual cylinder length=0.1 radius=0.1
- link wheel3: geometry collision cylinder length=0.1 radius=0.1; visual cylinder length=0.1 radius=0.1
- link wheel4: geometry collision cylinder length=0.1 radius=0.1; visual cylinder length=0.1 radius=0.1
Joints:
- joint joint_wheel1: limit effort=10000 velocity=1000 -> (none); origin xyz=0.25 -0.30 0.2 rpy=0 0 0 -> xyz=0.25 -0.30 0 rpy=0 0 0
- joint joint_wheel2: limit effort=10000 velocity=1000 -> (none); origin xyz=0.25 0.30 0.2 rpy=0 0 0 -> xyz=0.25 0.30 0 rpy=0 0 0
- joint joint_wheel3: limit effort=10000 velocity=1000 -> (none); origin xyz=-0.25 -0.30 0.2 rpy=0 0 0 -> xyz=-0.25 -0.30 0 rpy=0 0 0
- joint joint_wheel4: limit effort=10000 velocity=1000 -> (none); origin xyz=-0.25 0.30 0.2 rpy=0 0 0 -> xyz=-0.25 0.30 0 rpy=0 0 0
